Commit message: repo cleanup

File: src/test/urdf/robot.urdf (robot description, URDF)
Before this commit: robot test_robot, 1 links, 0 joints
Links:
- removed link Base link
- added link base_link; visual box size=0.5 0.5 0.5

Commit message: BBBB

File: src/test/urdf/robot.urdf (robot description, URDF)
Before this commit: robot test_robot, 1 links, 0 joints
Links:
- added link gripper_base, mass 1.0; collision box size=0.1 0.04 0.04; visual box size=0.1 0.04 0.04
- added link left_gripper_jaw, mass 1.0; collision box size=0.01 0.02 0.06; visual box size=0.01 0.02 0.06
- added link link_2, mass 1.0; collision box size=0.08 0.08 0.5; visual box size=0.08 0.08 0.5
- added link link_3, mass 1.0; collision box size=0.06 0.06 0.4; visual box size=0.06 0.06 0.4
- link base_link: mass None -> 1.0; geometry collision cylinder length=0.2 radius=0.1; visual cylinder length=0.2 radius=0.1
Joints:
- added joint gripper_base_joint: type fixed, parent link_3, child gripper_base, origin xyz=0 0 0.4 rpy=0 0 0
- added joint joint_1: type revolute, parent base_link, child link_2, origin xyz=0 0 0.1 rpy=0 0 0, axis 0 0 1, limit lower=-3.14 upper=3.14 effort=10.0 velocity=1.0
- added joint joint_2: type revolute, parent link_2, child link_3, origin xyz=0 0 0.5 rpy=0 0 0, axis 0 1 0, limit lower=-1.57 upper=1.57 effort=10.0 velocity=1.0
- added joint left_gripper_joint: type prismatic, parent gripper_base, child left_gripper_jaw, origin xyz=-0.04 0 0.02 rpy=0 0 0, axis 1 0 0, limit lower=0.0 upper=0.03 effort=5.0 velocity=0.5
